Commit message: Adds IMU, LiDAR and realsense camera plugins

File: via_robot/via_description/urdf/via.gazebo.xacro (robot description, xacro)
@@ -85,4 +85,75 @@
     </joint>
   </transmission>
+  <!-- IMU sensor -->
+  <gazebo reference="imu_link">
+    <sensor type="imu" name="imu">
+      <always_on>true</always_on>
+      <visualize>true</visualize>
+    </sensor>
+    <material>Gazebo/Green</material>
+  </gazebo>
+  <!-- IMU plugin -->
+  <gazebo>
+    <plugin name="imu_plugin" filename="libgazebo_ros_imu.so">
+      <alwaysOn>true</alwaysOn>
+      <bodyName>imu_link</bodyName>
+      <frameName>imu_link</frameName>
+      <topicName>imu</topicName>
+      <serviceName>imu_service</serviceName>
+      <gaussianNoise>0.0</gaussianNoise>
+      <updateRate>200</updateRate>
+      <imu>
+        <noise>
+          <type>gaussian</type>
+          <rate>
+            <mean>0.0</mean>
+            <stddev>2e-4</stddev>
+            <bias_mean>0.0000075</bias_mean>
+            <bias_stddev>0.0000008</bias_stddev>
+          </rate>
+          <accel>
+            <mean>0.0</mean>
+            <stddev>1.7e-2</stddev>
+            <bias_mean>0.1</bias_mean>
+            <bias_stddev>0.001</bias_stddev>
+          </accel>
+        </noise>
+      </imu>
+    </plugin>
+  </gazebo>
+  <!-- Hokuyo LiDAR -->
+  <gazebo reference="laser_frame">
+    <material>Gazebo/Red</material>
+    <sensor type="ray" name="head_hokuyo_sensor">
+      <pose>0 0 0 0 0 0</pose>
+      <visualize>true</visualize>
+      <update_rate>10</update_rate>
+      <ray>
+        <scan>
+          <horizontal>
+            <samples>360</samples>
+            <resolution>1</resolution>
+            <min_angle>-1.570796</min_angle>
+            <max_angle>1.570796</max_angle>
+          </horizontal>
+        </scan>
+        <range>
+          <min>0.3</min>
+          <max>10.0</max>
+          <resolution>0.01</resolution>
+        </range>
+        <noise>
+          <type>gaussian</type>
+          <mean>0.0</mean>
+          <stddev>0.01</stddev>
+        </noise>
+      </ray>
+      <plugin name="laser_controller" filename="libgazebo_ros_laser.so">
+        <topicName>/scan</topicName>
+        <frameName>laser_frame</frameName>
+        <!--output_type>sensor_msgs/LaserScan</output_type-->
+      </plugin>
+    </sensor>
+  </gazebo>
   <!-- Gazebo plugin for ROS Control -->
   <gazebo>

File: via_robot/via_description/urdf/via.urdf.xacro (robot description, xacro)
@@ -3,4 +3,5 @@
   <!-- Include gabezo tags for simulation -->
   <xacro:include filename="$(find via_description)/urdf/via.gazebo.xacro"/>
+	<xacro:include filename="$(find via_description)/urdf/d435/d435.urdf.xacro"/>
   <!-- Dummy base link, because KDL cannot have inertia on the base link -->
   <link name="base_footprint"/>
@@ -266,3 +267,50 @@
       velocity="10" />
   </joint>
+  <!--LIDAR Sensor-->
+  <link name="laser_frame">
+    <visual>
+      <geometry>
+        <mesh filename="package://via_description/meshes/sensors/hokuyo.dae"/>
+      </geometry>
+      <material name="red"/>
+    </visual>
+    <collision>
+      <geometry>
+        <mesh filename="package://via_description/meshes/sensors/hokuyo.dae"/>
+      </geometry>
+    </collision>
+    <inertial>
+      <mass value="0.114" />
+      <origin xyz="0 0 -0.03" />
+      <inertia ixx="0.001" ixy="0.0" ixz="0.0"
+               iyy="0.001" iyz="0.0"
+               izz="0.001" />
+    </inertial>
+  </link>
+  <joint name="laser_joint" type="fixed">
+    <parent link="base_link"/>
+    <child link="laser_frame"/>
+    <origin xyz="0.32 0.0 0.4" rpy="0 0 0"/>
+  </joint>
+	<!-- IMU -->
+  <joint name="imu_joint" type="fixed">
+    <parent link="base_link"/>
+    <child link="imu_link"/>
+    <origin xyz="0.06 0 0.35" rpy="0 0 0"/>
+  </joint>
+  <link name="imu_link">
+    <visual>
+      <origin xyz="0 0 0" rpy="0 0 0"/>
+      <geometry>
+        <box size="0.1 0.1 0.05"/>
+      </geometry>
+      <material name="">
+				<color rgba="0.8 0.0 0.0 1.0"/>
+			</material>
+    </visual>
+  </link>
+  <!-- Realsense Camera -->
+  <xacro:sensor_d435 name="realsense_d435" topics_ns="realsense_d435" parent="base_link">
+    <origin xyz="0.3 0 0.5" rpy="0 0.7854 0"/>
+  </xacro:sensor_d435>
 </robot>

Commit message: Add navigation framework for the via robot. EKF localization, map server, obstacle avoidance, with and without a map.

File: via_robot/via_description/urdf/via.gazebo.xacro (robot description, xacro)
@@ -134,6 +134,6 @@
             <samples>360</samples>
             <resolution>1</resolution>
-            <min_angle>-1.570796</min_angle>
-            <max_angle>1.570796</max_angle>
+            <min_angle>-3.1416</min_angle>
+            <max_angle>3.1416</max_angle>
           </horizontal>
         </scan>

File: via_robot/via_description/urdf/via.urdf.xacro (robot description, xacro)
@@ -291,7 +291,7 @@
     <parent link="base_link"/>
     <child link="laser_frame"/>
-    <origin xyz="0.32 0.0 0.4" rpy="0 0 0"/>
-  </joint>
-	<!-- IMU -->
+    <origin xyz="0.0 0.0 0.43" rpy="0 0 0"/>
+  </joint>
+  <!-- IMU -->
   <joint name="imu_joint" type="fixed">
     <parent link="base_link"/>
@@ -310,7 +310,11 @@
     </visual>
   </link>
-  <!-- Realsense Camera -->
-  <xacro:sensor_d435 name="realsense_d435" topics_ns="realsense_d435" parent="base_link">
-    <origin xyz="0.3 0 0.5" rpy="0 0.7854 0"/>
+  <!-- Realsense Front Camera -->
+  <xacro:sensor_d435 name="front_camera" topics_ns="front_camera" parent="base_link">
+    <origin xyz="0.3 0 0.55" rpy="0 0.5236 0"/>
+  </xacro:sensor_d435>
+    <!-- Realsense Back Camera -->
+  <xacro:sensor_d435 name="back_camera" topics_ns="back_camera" parent="base_link">
+    <origin xyz="-0.3 0 0.55" rpy="0 0.5236 3.1416"/>
   </xacro:sensor_d435>
 </robot>

Commit message: urdf atualized

File: via_robot/via_description/urdf/via.gazebo.xacro (robot description, xacro)
@@ -85,75 +85,4 @@
     </joint>
   </transmission>
-  <!-- IMU sensor -->
-  <gazebo reference="imu_link">
-    <sensor type="imu" name="imu">
-      <always_on>true</always_on>
-      <visualize>true</visualize>
-    </sensor>
-    <material>Gazebo/Green</material>
-  </gazebo>
-  <!-- IMU plugin -->
-  <gazebo>
-    <plugin name="imu_plugin" filename="libgazebo_ros_imu.so">
-      <alwaysOn>true</alwaysOn>
-      <bodyName>imu_link</bodyName>
-      <frameName>imu_link</frameName>
-      <topicName>imu</topicName>
-      <serviceName>imu_service</serviceName>
-      <gaussianNoise>0.0</gaussianNoise>
-      <updateRate>200</updateRate>
-      <imu>
-        <noise>
-          <type>gaussian</type>
-          <rate>
-            <mean>0.0</mean>
-            <stddev>2e-4</stddev>
-            <bias_mean>0.0000075</bias_mean>
-            <bias_stddev>0.0000008</bias_stddev>
-          </rate>
-          <accel>
-            <mean>0.0</mean>
-            <stddev>1.7e-2</stddev>
-            <bias_mean>0.1</bias_mean>
-            <bias_stddev>0.001</bias_stddev>
-          </accel>
-        </noise>
-      </imu>
-    </plugin>
-  </gazebo>
-  <!-- Hokuyo LiDAR -->
-  <gazebo reference="laser_frame">
-    <material>Gazebo/Red</material>
-    <sensor type="ray" name="head_hokuyo_sensor">
-      <pose>0 0 0 0 0 0</pose>
-      <visualize>false</visualize>
-      <update_rate>10</update_rate>
-      <ray>
-        <scan>
-          <horizontal>
-            <samples>360</samples>
-            <resolution>1</resolution>
-            <min_angle>-3.1416</min_angle>
-            <max_angle>3.1416</max_angle>
-          </horizontal>
-        </scan>
-        <range>
-          <min>0.3</min>
-          <max>20.0</max>
-          <resolution>0.01</resolution>
-        </range>
-        <noise>
-          <type>gaussian</type>
-          <mean>0.0</mean>
-          <stddev>0.01</stddev>
-        </noise>
-      </ray>
-      <plugin name="laser_controller" filename="libgazebo_ros_laser.so">
-        <topicName>/scan</topicName>
-        <frameName>laser_frame</frameName>
-        <!--output_type>sensor_msgs/LaserScan</output_type-->
-      </plugin>
-    </sensor>
-  </gazebo>
   <!-- Gazebo plugin for ROS Control -->
   <gazebo>

File: via_robot/via_description/urdf/via.urdf.xacro (robot description, xacro)
@@ -4,4 +4,6 @@
   <xacro:include filename="$(find via_description)/urdf/via.gazebo.xacro"/>
 	<xacro:include filename="$(find via_description)/urdf/d435/d435.urdf.xacro"/>
+  <xacro:include filename="$(find via_description)/urdf/LIDAR/lidar_hokuyo.urdf.xacro"/>
+  <xacro:include filename="$(find via_description)/urdf/IMU/imu.urdf.xacro"/>
   <xacro:include filename="$(find via_description)/urdf/gps/gps.xacro"/>
   <!-- Dummy base link, because KDL cannot have inertia on the base link -->
@@ -269,55 +271,16 @@
   </joint>
   <!--LIDAR Sensor-->
-  <link name="laser_frame">
-    <visual>
-      <geometry>
-        <mesh filename="package://via_description/meshes/sensors/hokuyo.dae"/>
-      </geometry>
-      <material name="red"/>
-    </visual>
-    <collision>
-      <geometry>
-        <mesh filename="package://via_description/meshes/sensors/hokuyo.dae"/>
-      </geometry>
-    </collision>
-    <inertial>
-      <mass value="0.114" />
-      <origin xyz="0 0 -0.03" />
-      <inertia ixx="0.001" ixy="0.0" ixz="0.0"
-               iyy="0.001" iyz="0.0"
-               izz="0.001" />
-    </inertial>
-  </link>
-  <joint name="laser_joint" type="fixed">
-    <parent link="base_link"/>
-    <child link="laser_frame"/>
-    <origin xyz="0.0 0.0 0.43" rpy="0 0 0"/>
-  </joint>
+  <!-- <xacro:lidar laser="lidar_hokuyo"/> -->
   <!-- IMU -->
-  <joint name="imu_joint" type="fixed">
-    <parent link="base_link"/>
-    <child link="imu_link"/>
-    <origin xyz="0.06 0 0.35" rpy="0 0 0"/>
-  </joint>
-  <link name="imu_link">
-    <visual>
-      <origin xyz="0 0 0" rpy="0 0 0"/>
-      <geometry>
-        <box size="0.1 0.1 0.05"/>
-      </geometry>
-      <material name="">
-				<color rgba="0.8 0.0 0.0 1.0"/>
-			</material>
-    </visual>
-  </link>
+  <xacro:imu sensor="imu"/>
   <!-- Realsense Front Camera -->
-  <xacro:sensor_d435 name="front_camera" topics_ns="front_camera" parent="base_link">
+  <!-- <xacro:sensor_d435 name="front_camera" topics_ns="front_camera" parent="base_link">
     <origin xyz="0.3 0 0.55" rpy="0 0.5236 0"/>
-  </xacro:sensor_d435>
-    <!-- Realsense Back Camera -->
-  <xacro:sensor_d435 name="back_camera" topics_ns="back_camera" parent="base_link">
+  </xacro:sensor_d435> -->
+  <!-- Realsense Back Camera -->
+  <!-- <xacro:sensor_d435 name="back_camera" topics_ns="back_camera" parent="base_link">
     <origin xyz="-0.3 0 0.55" rpy="0 0.5236 3.1416"/>
-  </xacro:sensor_d435>
-    <!-- GPS -->
-    <xacro:gps joint="joint_chassis_gps" link="link_gps" parent="base_link" height1="0.2" width="0.02" lat_origin="-22.004127333333333" long_origin="-47.93340416666667" alt_origin="829"/>
+  </xacro:sensor_d435> -->
+  <!-- GPS -->
+  <xacro:gps joint="joint_chassis_gps" link="link_gps" parent="base_link" height1="0.2" width="0.02" lat_origin="-22.004127333333333" long_origin="-47.93340416666667" alt_origin="829"/>
 </robot>
